File: pcbs/blow_button_board/blow_button_board.kicad_pcb (KiCad board)
At the start: 2 copper layers, 14 x 17 mm, 2 parts, among them J1 Conn_01x02_Pin, SW1 SW_Push

Commit message: Update PCBs
Other:
- board text added: "blow board"
- board text added: "v0.1"
