File: pcbs/valves_board/valves_board.kicad_pcb (KiCad board)
At the start: 2 copper layers, 68 x 13 mm, 4 parts, among them J1 mainboard_connector, SW1 SW_Push, SW2 SW_Push, SW3 SW_Push

Commit message: Update PCBs
Other:
- board text added: "gnd"
- board text added: "v0.1"
- board text added: "valve board"
- board text added: "vl1"
- board text added: "vl2"
- board text added: "vl3"
