File: pcbs/trumpet_synth_mainboard/trumpet_synth_mainboard.kicad_pcb (KiCad board)
At the start: 2 copper layers, 76.6 x 82.5 mm, 15 parts, among them J1 valve_board_connector, J2 blow_board_connector, J3 Power, J4 SWD, J5 i2c_breakout, SW1 SW_Push, U1 Pico

Commit message: Update PCBs
Parts:
- moved J4 5.90 mm to (74.0, 65.0), turned to 90 degrees
- moved SW1 3.00 mm to (49.0, 65.0)
- moved J3 0.73 mm to (95.0, 63.7)
Routing:
- net Net-(J4-Pin_3): track 21.9 -> 14.4 mm
- net Net-(J4-Pin_1): track 23.0 -> 29.6 mm
- net +5V: track 115.2 -> 113.8 mm, vias 1 -> 0
- net Net-(J4-Pin_2): track 22.2 -> 23.0 mm
Changed lines of the file:
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@@
 	)
 	(footprint "Connector_PinHeader_2.54mm:PinHeader_1x03_P2.54mm_Vertical"
+		(locked yes)
 		(layer "F.Cu")
-		(at 48.96 62 90)
+		(at 48.96 65 90)
 		(descr "Through hole straight pin header, 1x03, 2.54mm pitch, single row")
 		(tags "Through hole pin header THT 1x03 2.54mm single row")
@@
 	)
 	(footprint "Connector_PinHeader_2.54mm:PinHeader_1x03_P2.54mm_Vertical"
+		(locked yes)
 		(layer "F.Cu")
-		(at 79.04 62 -90)
+		(at 73.96 65 90)
 		(descr "Through hole straight pin header, 1x03, 2.54mm pitch, single row")
 		(tags "Through hole pin header THT 1x03 2.54mm single row")
@@
 		(attr through_hole)
 		(fp_line
-			(start -1.38 6.46)
-			(end 1.38 6.46)
+			(start -1.38 -1.38)
+			(end 0 -1.38)
 			(stroke
 				(width 0.12)
@@
 		)
 		(fp_line
-			(start -1.38 1.27)
-			(end -1.38 6.46)
+			(start -1.38 0)
+			(end -1.38 -1.38)
 			(stroke
 				(width 0.12)
@@
 		)
 		(fp_line
-			(start -1.38 1.27)
-			(end 1.38 1.27)
+			(start 1.38 1.27)
+			(end 1.38 6.46)
 			(stroke
 				(width 0.12)
@@
 		)
 		(fp_line
-			(start 1.38 1.27)
-			(end 1.38 6.46)
+			(start -1.38 1.27)
+			(end 1.38 1.27)
 			(stroke
 				(width 0.12)
@@
 		)
 		(fp_line
-			(start -1.38 0)
-			(end -1.38 -1.38)
+			(start -1.38 1.27)
+			(end -1.38 6.46)
 			(stroke
 				(width 0.12)
@@
 		)
 		(fp_line
-			(start -1.38 -1.38)
-			(end 0 -1.38)
+			(start -1.38 6.46)
+			(end 1.38 6.46)
 			(stroke
 				(width 0.12)
@@
 		)
 		(fp_line
-			(start -1.77 6.85)
-			(end 1.77 6.85)
+			(start 1.77 -1.77)
+			(end -1.77 -1.77)
 			(stroke
 				(width 0.05)
@@
 		)
 		(fp_line
-			(start 1.77 6.85)
-			(end 1.77 -1.77)
+			(start -1.77 -1.77)
+			(end -1.77 6.85)
 			(stroke
 				(width 0.05)
@@
 		)
 		(fp_line
-			(start -1.77 -1.77)
-			(end -1.77 6.85)
+			(start 1.77 6.85)
+			(end 1.77 -1.77)
 			(stroke
 				(width 0.05)
@@
 		)
 		(fp_line
-			(start 1.77 -1.77)
-			(end -1.77 -1.77)
+			(start -1.77 6.85)
+			(end 1.77 6.85)
 			(stroke
 				(width 0.05)
@@
 		)
 		(fp_line
-			(start -1.27 6.35)
-			(end -1.27 -0.635)
+			(start 1.27 -1.27)
+			(end 1.27 6.35)
 			(stroke
 				(width 0.1)
@@
 		)
 		(fp_line
-			(start 1.27 6.35)
-			(end -1.27 6.35)
+			(start -0.635 -1.27)
+			(end 1.27 -1.27)
 			(stroke
 				(width 0.1)
@@
 		)
 		(fp_line
-			(start -0.635 -1.27)
-			(end 1.27 -1.27)
+			(start 1.27 6.35)
+			(end -1.27 6.35)
 			(stroke
 				(width 0.1)
@@
 		)
 		(fp_line
-			(start 1.27 -1.27)
-			(end 1.27 6.35)
+			(start -1.27 6.35)
+			(end -1.27 -0.635)
 			(stroke
 				(width 0.1)
@@
 		)
 		(pad "1" thru_hole rect
-			(at 0 0 270)
+			(at 0 0 90)
 			(size 1.7 1.7)
 			(drill 1)
@@
 		)
 		(pad "2" thru_hole circle
-			(at 0 2.54 270)
+			(at 0 2.54 90)
 			(size 1.7 1.7)
 			(drill 1)
@@
 		)
 		(pad "3" thru_hole circle
-			(at 0 5.08 270)
+			(at 0 5.08 90)
 			(size 1.7 1.7)
 			(drill 1)
@@
 	(footprint "Connector_PinHeader_2.54mm:PinHeader_1x02_P2.54mm_Vertical"
 		(layer "F.Cu")
-		(at 95 63)
+		(at 95 63.725)
 		(descr "Through hole straight pin header, 1x02, 2.54mm pitch, single row")
 		(tags "Through hole pin header THT 1x02 2.54mm single row")
@@
 	)
 	(segment
-		(start 45.96 65)
-		(end 48 65)
-		(width 0.35)
-		(layer "F.Cu")
-		(net 5)
-	)
-	(segment
-		(start 34.41 69.8)
-		(end 34.41 67.59)
-		(width 0.35)
-		(layer "F.Cu")
-		(net 5)
-	)
-	(segment
 		(start 37 65)
-		(end 45.96 65)
+		(end 48.96 65)
 		(width 0.35)
 		(layer "F.Cu")
@@
 	)
 	(segment
-		(start 45.96 65)
-		(end 48.96 62)
+		(start 34.41 69.8)
+		(end 34.41 67.59)
 		(width 0.35)
 		(layer "F.Cu")
 		(net 5)
 	)
-	(via
-		(at 48 65)
-		(size 0.6)
-		(drill 0.3)
-		(layers "F.Cu" "B.Cu")
+	(segment
+		(start 80 85)
+		(end 77 82)
+		(width 0.35)
+		(layer "B.Cu")
 		(net 5)
 	)
 	(segment
-		(start 80 85)
+		(start 96.894 91.894)
 		(end 90 85)
 		(width 0.35)
@@
 	)
 	(segment
-		(start 77 82)
-		(end 80 85)
+		(start 65.5 61.5)
+		(end 52.46 61.5)
 		(width 0.35)
 		(layer "B.Cu")
@@
 	)
 	(segment
-		(start 96.894 91.894)
-		(end 96.894 120.65)
+		(start 52.46 61.5)
+		(end 48.96 65)
 		(width 0.35)
 		(layer "B.Cu")
@@
 	)
 	(segment
-		(start 69 65)
-		(end 77 73)
+		(start 77 73)
+		(end 65.5 61.5)
 		(width 0.35)
 		(layer "B.Cu")
@@
 	)
 	(segment
-		(start 48 65)
-		(end 69 65)
+		(start 90 85)
+		(end 80 85)
 		(width 0.35)
 		(layer "B.Cu")
@@
 	)
 	(segment
-		(start 77 73)
-		(end 77 82)
+		(start 77 82)
+		(end 77 73)
 		(width 0.35)
 		(layer "B.Cu")
@@
 	)
 	(segment
-		(start 90 85)
+		(start 96.894 120.65)
 		(end 96.894 91.894)
 		(width 0.35)
@@
 	)
 	(segment
-		(start 89 63)
-		(end 95 63)
+		(start 91 62)
+		(end 92.725 63.725)
 		(width 0.35)
 		(layer "F.Cu")
@@
 	)
 	(segment
-		(start 87 65)
-		(end 89 63)
+		(start 92.725 63.725)
+		(end 95 63.725)
 		(width 0.35)
 		(layer "F.Cu")
@@
 	)
 	(segment
-		(start 51.5 62)
-		(end 54.5 65)
+		(start 54.5 62)
+		(end 91 62)
 		(width 0.35)
 		(layer "F.Cu")
@@
 	)
 	(segment
-		(start 54.5 65)
-		(end 87 65)
+		(start 51.5 65)
+		(end 54.5 62)
 		(width 0.35)
 		(layer "F.Cu")
@@
 	)
 	(segment
-		(start 83 75.59)
-		(end 83 67.4329)
-		(width 0.2)
-		(layer "B.Cu")
-		(net 19)
-	)
-	(segment
-		(start 80.5671 65)
-		(end 78 65)
-		(width 0.2)
-		(layer "B.Cu")
-		(net 19)
-	)
-	(segment
-		(start 78 65)
-		(end 76.5 63.5)
+		(start 78 63.5)
+		(end 76.5 65)
 		(width 0.2)
 		(layer "B.Cu")
@@
 	)
 	(segment
-		(start 76.5 63.5)
-		(end 76.5 62)
+		(start 83 64.5)
+		(end 82 63.5)
 		(width 0.2)
 		(layer "B.Cu")
@@
 	)
 	(segment
-		(start 83 67.4329)
-		(end 80.5671 65)
+		(start 82 63.5)
+		(end 78 63.5)
 		(width 0.2)
 		(layer "B.Cu")
@@
 	)
 	(segment
-		(start 79.9 76.15)
-		(end 82 74.05)
-		(width 0.2)
-		(layer "B.Cu")
-		(net 20)
-	)
-	(segment
-		(start 73.96 64.96)
-		(end 73.96 62)
+		(start 83 75.59)
+		(end 83 64.5)
 		(width 0.2)
 		(layer "B.Cu")
-		(net 20)
+		(net 19)
 	)
 	(segment
 		(start 82 74.05)
-		(end 82 67)
+		(end 82 66)
 		(width 0.2)
 		(layer "B.Cu")
@@
 	)
 	(segment
-		(start 81 66)
-		(end 75 66)
+		(start 81 65)
+		(end 82 66)
 		(width 0.2)
 		(layer "B.Cu")
@@
 	)
 	(segment
-		(start 82 67)
-		(end 81 66)
+		(start 79.9 76.15)
+		(end 82 74.05)
 		(width 0.2)
 		(layer "B.Cu")
@@
 	)
 	(segment
-		(start 75 66)
-		(end 73.96 64.96)
+		(start 81 65)
+		(end 79.04 65)
 		(width 0.2)
 		(layer "B.Cu")
@@
 	)
 	(segment
-		(start 79.9 81.23)
-		(end 84 77.13)
+		(start 75.861 63.099)
+		(end 73.96 65)
 		(width 0.2)
 		(layer "B.Cu")
@@
 	)
 	(segment
-		(start 80.0671 63.0271)
-		(end 79.04 62)
+		(start 79.9 81.23)
+		(end 84 77.13)
 		(width 0.2)
 		(layer "B.Cu")
@@
 	)
 	(segment
-		(start 84 67.8658)
-		(end 80.0671 63.9329)
+		(start 82.1661 63.099)
+		(end 75.861 63.099)
 		(width 0.2)
 		(layer "B.Cu")
@@
 	)
 	(segment
-		(start 80.0671 63.9329)
-		(end 80.0671 63.0271)
+		(start 84 64.9329)
+		(end 82.1661 63.099)
 		(width 0.2)
 		(layer "B.Cu")
@@
 	(segment
 		(start 84 77.13)
-		(end 84 67.8658)
+		(end 84 64.9329)
 		(width 0.2)
 		(layer "B.Cu")

Commit message: Order all PCBs v0.1
Parts:
- removed J3: Power, Connector_PinHeader_2.54mm:PinHeader_1x02_P2.54mm_Vertical
- added J6: Conn_01x03_Pin, Connector_PinHeader_2.54mm:PinHeader_1x03_P2.54mm_Vertical, F.Cu at (95.0, 63.5)
Connections:
- SW1 pad 1: +5V -> Net-(J6-Pin_3)
- SW1 pad 2: Net-(J3-Pin_1) -> GND
Routing:
- net Net-(J6-Pin_3): track 0.00 -> 50.4 mm
- net Net-(J3-Pin_1): track 45.5 -> 0.00 mm
- net +5V: track 113.8 -> 124.3 mm, vias 0 -> 1
- net /GPIO0: track 102.8 -> 106.5 mm
- net /GPIO6: track 76.8 -> 78.0 mm
- net /GPIO9: track 77.5 -> 76.7 mm
- net /GPIO22: track 118.3 -> 117.5 mm
Other:
- board text added: "+5V"
- board text added: "EN"
- board text added: "GND"
