File: pcbs/trumpet_synth_mainboard/trumpet_synth_mainboard.kicad_sch (KiCad schematic)
At the start: 15 parts, among them J1 valve_board_connector, J2 blow_board_connector, J3 Power, J4 SWD, J5 i2c_breakout, SW1 SW_Push, U1 Pico

Commit message: Update PCBs
Other:
- note added: "TODO: x make SWD pins accessible from case x make power switch accessible from case x double check linpot pins used x jack footprint is wrong"
- note removed: "TODO: - make SWD pins accessible from case - make power switch accessible from case - double check linpot pins used x jack footprint is wrong"
Changed lines of the file:
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@@
 	(generator_version "9.0")
 	(paper "A4")
-	(text "TODO:\n- make SWD pins accessible from case\n- make power switch accessible from case\n- double check linpot pins used\nx jack footprint is wrong"
+	(text "TODO:\nx make SWD pins accessible from case\nx make power switch accessible from case\nx double check linpot pins used\nx jack footprint is wrong"
 		(exclude_from_sim no)
 		(at 187.452 21.844 0)

Commit message: Order all PCBs v0.1
Parts:
- removed J3: Power, Connector_PinHeader_2.54mm:PinHeader_1x02_P2.54mm_Vertical, symbol Connector:Conn_01x02_Pin
- added J6: Conn_01x03_Pin, Connector_PinHeader_2.54mm:PinHeader_1x03_P2.54mm_Vertical, symbol Connector:Conn_01x03_Pin
Connections:
- net +5V: now also J6.2 (Pin_2); no longer SW1.1
- net GND: now also SW1.2, J6.1 (Pin_1)
- new net: J6.3 (Pin_3), SW1.1
Other:
- note added: "TODO: x make SWD pins accessible from case x make power switch accessible from case x double check linpot pins used x jack footprint is wrong - make 3 power pins available from case"
- note removed: "TODO: x make SWD pins accessible from case x make power switch accessible from case x double check linpot pins used x jack footprint is wrong"
- moved on the sheet: SW1

Commit message: Tests on PCB
Other:
- note added: "TODO: x make SWD pins accessible from case x make power switch accessible from case x double check linpot pins used x jack footprint is wrong x make 3 power pins available from case - use headers for board to board connections (directly soldered on wires break) and make sure the case has space for them - got lucky with DAC placement, 3.5mm jack could've collided with the linear pot - use a differ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"
- note removed: "TODO: x make SWD pins accessible from case x make power switch accessible from case x double check linpot pins used x jack footprint is wrong - make 3 power pins available from case"
Changed lines of the file:
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@@
 	(generator_version "9.0")
 	(paper "A4")
-	(text "TODO:\nx make SWD pins accessible from case\nx make power switch accessible from case\nx double check linpot pins used\nx jack footprint is wrong\n- make 3 power pins available from case"
+	(text "TODO:\nx make SWD pins accessible from case\nx make power switch accessible from case\nx double check linpot pins used\nx jack footprint is wrong\nx make 3 power pins available from case\n- use headers for board to board connections (directly soldered on wires break) and make sure the case has space for them\n- got lucky with DAC placement, 3.5mm jack could've collided with the linear pot\n- use a different RGB LED footprint, this one is to error prone to solder"
 		(exclude_from_sim no)
 		(at 187.452 21.844 0)
